Commit message: dev: fix primitives config

File: source/BipeD/BipeD/assets/BD_asset/BD_prims.urdf (robot description, URDF)
Before this commit: robot BD, 11 links, 10 joints
Links:
- link L0_Link: geometry visual mesh filename=./meshes/L0_Link.STL
- link L1_Link: geometry visual mesh filename=./meshes/L1_Link.STL
- link R0_Link: geometry visual mesh filename=./meshes/R0_Link.STL
- link R1_Link: geometry visual mesh filename=./meshes/R1_Link.STL

Commit message: dev: fix? collision (prims), add versions to readme

File: source/BipeD/BipeD/assets/BD_asset/BD_prims.urdf (robot description, URDF)
Before this commit: robot BD, 11 links, 10 joints
Links:
- link L2_Link: geometry collision cylinder length=0.120 radius=0.02; visual mesh filename=./meshes/L2_Link.STL
- link L4_Link_ankle: geometry collision box size=0.14 0.050 0.018; visual mesh filename=./meshes/L4_Link_ankle.STL
- link R2_Link: geometry collision cylinder length=0.120 radius=0.02; visual mesh filename=./meshes/R2_Link.STL
- link R4_Link_ankle: geometry collision box size=0.14 0.050 0.018; visual mesh filename=./meshes/R4_Link_ankle.STL
- link base_link: geometry collision box size=0.12 0.16 0.12; visual mesh filename=./meshes/base_link.STL

Commit message: feat: update ranges

File: source/BipeD/BipeD/assets/BD_asset/BD_prims.urdf (robot description, URDF)
Before this commit: robot BD, 11 links, 10 joints
Joints:
- joint J_L3: limit lower=-2.35 upper=0.05 effort=20 velocity=20 -> lower=-1.57 upper=0.05 effort=20 velocity=20
- joint J_L4_ankle: limit lower=-0.6 upper=0.7 effort=12 velocity=20 -> lower=-0.78 upper=0.7 effort=12 velocity=20
- joint J_R2: limit lower=-0.57 upper=1.57 effort=20 velocity=20 -> lower=-1.57 upper=0.57 effort=20 velocity=20
- joint J_R3: limit lower=-0.05 upper=2.35 effort=20 velocity=20 -> lower=-0.05 upper=1.57 effort=20 velocity=20
- joint J_R4_ankle: limit lower=-0.7 upper=0.6 effort=12 velocity=20 -> lower=-0.7 upper=0.78 effort=12 velocity=20

Commit message: fix: urdf model orientation and joints

File: source/BipeD/BipeD/assets/BD_asset/BD_prims.urdf (robot description, URDF)
Before this commit: robot BD, 11 links, 10 joints
Joints:
- joint J_L0: axis 0 0 1 -> 0 0 -1; origin xyz=0.0025357 0.053301 0.056145 rpy=0 0 0 -> xyz=0.0 0.053301 0.056145 rpy=0 0 3.14
- joint J_L2: origin xyz=0.010958 0.073699 -0.014313 rpy=0 0 0 -> xyz=0.010958 -0.073699 -0.014313 rpy=0 0 3.14
- joint J_L3: axis 0 1 0 -> 0 -1 0; limit lower=-1.57 upper=0.05 effort=20 velocity=20 -> lower=-0.1 upper=1.57 effort=20 velocity=20
- joint J_L4_ankle: axis 0 -1 0 -> 0 1 0; limit lower=-0.78 upper=0.7 effort=12 velocity=20 -> lower=-0.3 upper=0.8 effort=12 velocity=20
- joint J_R0: axis 0 0 1 -> 0 0 -1; origin xyz=0.0025357 -0.053425 0.056145 rpy=0 0 0 -> xyz=0.0 -0.053425 0.056145 rpy=0 0 3.14
- joint J_R2: origin xyz=0.010958 -0.073575 -0.014313 rpy=0 0 0 -> xyz=0.010958 0.073575 -0.014313 rpy=0 0 3.14
- joint J_R3: axis 0 -1 0 -> 0 1 0; limit lower=-0.05 upper=1.57 effort=20 velocity=20 -> lower=-1.57 upper=0.10 effort=20 velocity=20
- joint J_R4_ankle: axis 0 1 0 -> 0 -1 0; limit lower=-0.7 upper=0.78 effort=12 velocity=20 -> lower=-0.8 upper=0.3 effort=12 velocity=20
