Commit message: fix: collisions and inertia params, new usd 'BD'

File: source/BipeD/BipeD/assets/BD_asset/BD.urdf (robot description, URDF)
Before this commit: robot BD, 11 links, 10 joints
Links:
- link L0_Link: geometry visual mesh filename=./meshes/L0_Link.STL
- link L1_Link: mass 0.0295521887544817 -> 0.5; geometry visual mesh filename=./meshes/L1_Link.STL
- link L2_Link: mass 1.34863094594399 -> 0.5; geometry collision cylinder length=0.120 radius=0.02; visual mesh filename=./meshes/L2_Link.STL
- link L3_Link: mass 0.629727076499127 -> 0.5; geometry collision cylinder length=0.120 radius=0.022; visual mesh filename=./meshes/L3_Link.STL
- link L4_Link_ankle: mass 0.171742682777178 -> 0.15; geometry collision box size=0.14 0.050 0.018; visual mesh filename=./meshes/L4_Link_ankle.STL
- link R0_Link: geometry visual mesh filename=./meshes/R0_Link.STL
- link R1_Link: mass 0.029551251476222 -> 0.5; geometry visual mesh filename=./meshes/R1_Link.STL
- link R2_Link: mass 1.35023891621348 -> 0.5; geometry collision cylinder length=0.120 radius=0.02; visual mesh filename=./meshes/R2_Link.STL
- link R3_Link: mass 0.511661896307101 -> 0.5; geometry collision cylinder length=0.120 radius=0.022; visual mesh filename=./meshes/R3_Link.STL
- link R4_Link_ankle: mass 0.17174 -> 0.15; geometry collision box size=0.14 0.050 0.018; visual mesh filename=./meshes/R4_Link_ankle.STL
- link base_link: geometry collision box size=0.22 0.16 0.16; visual mesh filename=./meshes/base_link.STL
Joints:
- joint J_L0: axis 0 0 1 -> 0 0 -1; origin xyz=0.0025357 0.053301 0.056145 rpy=0 0 0 -> xyz=0.0 0.053301 0.056145 rpy=0 0 3.14
- joint J_L2: origin xyz=0.010958 0.073699 -0.014313 rpy=0 0 0 -> xyz=0.010958 -0.073699 -0.014313 rpy=0 0 3.14
- joint J_L3: axis 0 1 0 -> 0 -1 0; limit lower=-2.35 upper=0.05 effort=20 velocity=20 -> lower=-0.1 upper=1.57 effort=20 velocity=20
- joint J_L4_ankle: axis 0 -1 0 -> 0 1 0; limit lower=-0.6 upper=0.7 effort=12 velocity=20 -> lower=-0.3 upper=0.8 effort=12 velocity=20
- joint J_R0: axis 0 0 1 -> 0 0 -1; origin xyz=0.0025357 -0.053425 0.056145 rpy=0 0 0 -> xyz=0.0 -0.053425 0.056145 rpy=0 0 3.14
- joint J_R2: limit lower=-0.57 upper=1.57 effort=20 velocity=20 -> lower=-1.57 upper=0.57 effort=20 velocity=20; origin xyz=0.010958 -0.073575 -0.014313 rpy=0 0 0 -> xyz=0.010958 0.073575 -0.014313 rpy=0 0 3.14
- joint J_R3: axis 0 -1 0 -> 0 1 0; limit lower=-0.05 upper=2.35 effort=20 velocity=20 -> lower=-1.57 upper=0.10 effort=20 velocity=20
- joint J_R4_ankle: axis 0 1 0 -> 0 -1 0; limit lower=-0.7 upper=0.6 effort=12 velocity=20 -> lower=-0.8 upper=0.3 effort=12 velocity=20

File: source/BipeD/BipeD/assets/BD_asset/BD_old.urdf (robot description, URDF)
Before this commit: robot BD, 11 links, 10 joints
Links:
- link L0_Link: geometry collision mesh filename=./meshes/L0_Link.STL; visual mesh filename=./meshes/L0_Link.STL
- link L1_Link: geometry collision mesh filename=./meshes/L1_Link.STL; visual mesh filename=./meshes/L1_Link.STL
- link L2_Link: geometry collision mesh filename=./meshes/L2_Link.STL; visual mesh filename=./meshes/L2_Link.STL
- link L3_Link: geometry collision mesh filename=./meshes/L3_Link.STL; visual mesh filename=./meshes/L3_Link.STL
- link L4_Link_ankle: geometry collision mesh filename=./meshes/L4_Link_ankle.STL; visual mesh filename=./meshes/L4_Link_ankle.STL
- link R0_Link: geometry collision mesh filename=./meshes/R0_Link.STL; visual mesh filename=./meshes/R0_Link.STL
- link R1_Link: geometry collision mesh filename=./meshes/R1_Link.STL; visual mesh filename=./meshes/R1_Link.STL
- link R2_Link: geometry collision mesh filename=./meshes/R2_Link.STL; visual mesh filename=./meshes/R2_Link.STL
- link R3_Link: geometry collision mesh filename=./meshes/R3_Link.STL; visual mesh filename=./meshes/R3_Link.STL
- link R4_Link_ankle: geometry collision mesh filename=./meshes/R4_Link_ankle.STL; visual mesh filename=./meshes/R4_Link_ankle.STL
- link base_link: geometry collision mesh filename=./meshes/base_link.STL; visual mesh filename=./meshes/base_link.STL
Joints:
- joint J_L0: axis 0 0 -1 -> 0 0 1; origin xyz=0.0 0.053301 0.056145 rpy=0 0 3.14 -> xyz=0.0025357 0.053301 0.056145 rpy=0 0 0
- joint J_L2: origin xyz=0.010958 -0.073699 -0.014313 rpy=0 0 3.14 -> xyz=0.010958 0.073699 -0.014313 rpy=0 0 0
- joint J_L3: axis 0 -1 0 -> 0 1 0; limit lower=-0.1 upper=1.57 effort=20 velocity=20 -> lower=-2.35 upper=0.05 effort=20 velocity=20
- joint J_L4_ankle: axis 0 1 0 -> 0 -1 0; limit lower=-0.3 upper=0.8 effort=12 velocity=20 -> lower=-0.6 upper=0.7 effort=12 velocity=20
- joint J_R0: axis 0 0 -1 -> 0 0 1; origin xyz=0.0 -0.053425 0.056145 rpy=0 0 3.14 -> xyz=0.0025357 -0.053425 0.056145 rpy=0 0 0
- joint J_R2: limit lower=-1.57 upper=0.57 effort=20 velocity=20 -> lower=-0.57 upper=1.57 effort=20 velocity=20; origin xyz=0.010958 0.073575 -0.014313 rpy=0 0 3.14 -> xyz=0.010958 -0.073575 -0.014313 rpy=0 0 0
- joint J_R3: axis 0 1 0 -> 0 -1 0; limit lower=-1.57 upper=0.10 effort=20 velocity=20 -> lower=-0.05 upper=2.35 effort=20 velocity=20
- joint J_R4_ankle: axis 0 -1 0 -> 0 1 0; limit lower=-0.8 upper=0.3 effort=12 velocity=20 -> lower=-0.7 upper=0.6 effort=12 velocity=20

Commit message: dev: update cfg after model(urdf) changes

File: source/BipeD/BipeD/assets/BD_asset/BD.urdf (robot description, URDF)
Before this commit: robot BD, 11 links, 10 joints
Links:
- link L0_Link: mass 0.587331353457417 -> 0.55
- link L1_Link: mass 0.5 -> 0.55
- link L2_Link: mass 0.5 -> 0.55
- link L3_Link: mass 0.5 -> 0.35
- link R0_Link: mass 0.587331353381893 -> 0.55
- link R1_Link: mass 0.5 -> 0.55
- link R2_Link: mass 0.5 -> 0.55
- link R3_Link: mass 0.5 -> 0.35
- link base_link: mass 3 -> 2
